Commit message: rename joints and links in xacro

File: src/hexapod_model/urdf/hexapod.xacro (robot description, xacro)
@@ -37,5 +37,5 @@
 			</visual>
 		</link>
-		<link name="leg_${side}_${num}_f3">
+		<link name="leg_${side}_${num}_f2">
 			<visual>
 				<origin rpy="${1.5 * pi} 0 ${0.5 * pi}" xyz="0 -0.053 0.013"/>
@@ -54,5 +54,5 @@
 			</visual>
 		</link>
-		<link name="leg_${side}_${num}_f2">
+		<link name="leg_${side}_${num}_f3">
 			<visual>
 				<origin rpy="${1.5 * pi} 0 0" xyz="-0.063 0 0.013"/>
@@ -95,14 +95,14 @@
 			<limit lower="-${0.5 * pi}" upper="${0.5 * pi}" effort="15" velocity="1.0" />
 	  	</joint>
-		<joint name="joint_${side}_${num}_f3" type="revolute">
+		<joint name="joint_${side}_${num}_f2" type="revolute">
 			<parent link="leg_${side}_${num}_f1"/>
-			<child link="leg_${side}_${num}_f3"/>
+			<child link="leg_${side}_${num}_f2"/>
 			<origin xyz="0.062 0.0 0.0" rpy="0 0 ${0.5 * pi}" />
 			<axis xyz="1 0 0" />
 			<limit lower="-${0.5 * pi}" upper="${0.5 * pi}" effort="15" velocity="1.0" />
 	  	</joint>
-		<joint name="joint_${side}_${num}_f2" type="revolute">
-			<parent link="leg_${side}_${num}_f3"/>
-			<child link="leg_${side}_${num}_f2"/>
+		<joint name="joint_${side}_${num}_f3" type="revolute">
+			<parent link="leg_${side}_${num}_f2"/>
+			<child link="leg_${side}_${num}_f3"/>
 			<origin xyz="0.0 -0.094 0.0" rpy="0 -${0.32 * pi} ${0.5 * pi}" />
 			<axis xyz="0 1 0" />
@@ -110,5 +110,5 @@
 	  	</joint>
 		<joint name="joint_${side}_${num}_f4" type="revolute">
-			<parent link="leg_${side}_${num}_f2"/>
+			<parent link="leg_${side}_${num}_f3"/>
 			<child link="leg_${side}_${num}_f4"/>
 			<origin xyz="-0.104 0.0 0.0" rpy="-0 0 ${0.5 * pi}" />
