Commit message: update collision

File: src/hexapod_model/urdf/hexapod.urdf (robot description, URDF)
Before this commit: robot hexapod, 25 links, 24 joints
Links:
- removed link leg__1_f1
- removed link leg__1_f2
- removed link leg__1_f3
- removed link leg__1_f4
- added link leg_l_1_end; collision box size=0.02 0.005 0.02; visual box size=0.02 0.005 0.02
- added link leg_l_2_end; collision box size=0.02 0.005 0.02; visual box size=0.02 0.005 0.02
- added link leg_l_3_end; collision box size=0.02 0.005 0.02; visual box size=0.02 0.005 0.02
- added link leg_r_1_end; collision box size=0.02 0.005 0.02; visual box size=0.02 0.005 0.02
- added link leg_r_1_f1; collision box size=0.05 0.07 0.05; visual mesh filename=package://hexapod_model/meshes/femur_1_bin.stl
- added link leg_r_1_f2; collision box size=0.11 0.03 0.06; visual mesh filename=package://hexapod_model/meshes/femur_3_bin.stl
- added link leg_r_1_f3; collision box size=0.12 0.03 0.06; visual mesh filename=package://hexapod_model/meshes/femur_2_bin.stl
- added link leg_r_1_f4; collision box size=0.08 0.03 0.06; visual mesh filename=package://hexapod_model/meshes/femur_4_bin.stl
- added link leg_r_2_end; collision box size=0.02 0.005 0.02; visual box size=0.02 0.005 0.02
- added link leg_r_3_end; collision box size=0.02 0.005 0.02; visual box size=0.02 0.005 0.02
- link base_link: geometry collision box size=0.19 0.05 0.14; visual mesh filename=package://hexapod_model/meshes/body_bin.stl
- link leg_l_1_f1: geometry collision box size=0.05 0.07 0.05; visual mesh filename=package://hexapod_model/meshes/femur_1_bin.stl
- link leg_l_1_f2: geometry collision box size=0.11 0.03 0.06; visual mesh filename=package://hexapod_model/meshes/femur_3_bin.stl
- link leg_l_1_f3: geometry collision box size=0.12 0.03 0.06; visual mesh filename=package://hexapod_model/meshes/femur_2_bin.stl
- link leg_l_1_f4: geometry collision box size=0.08 0.03 0.06; visual mesh filename=package://hexapod_model/meshes/femur_4_bin.stl
- link leg_l_2_f1: geometry collision box size=0.05 0.07 0.05; visual mesh filename=package://hexapod_model/meshes/femur_1_bin.stl
- link leg_l_2_f2: geometry collision box size=0.11 0.03 0.06; visual mesh filename=package://hexapod_model/meshes/femur_3_bin.stl
- link leg_l_2_f3: geometry collision box size=0.12 0.03 0.06; visual mesh filename=package://hexapod_model/meshes/femur_2_bin.stl
- link leg_l_2_f4: geometry collision box size=0.08 0.03 0.06; visual mesh filename=package://hexapod_model/meshes/femur_4_bin.stl
- link leg_l_3_f1: geometry collision box size=0.05 0.07 0.05; visual mesh filename=package://hexapod_model/meshes/femur_1_bin.stl
- link leg_l_3_f2: geometry collision box size=0.11 0.03 0.06; visual mesh filename=package://hexapod_model/meshes/femur_3_bin.stl
- link leg_l_3_f3: geometry collision box size=0.12 0.03 0.06; visual mesh filename=package://hexapod_model/meshes/femur_2_bin.stl
- link leg_l_3_f4: geometry collision box size=0.08 0.03 0.06; visual mesh filename=package://hexapod_model/meshes/femur_4_bin.stl
- link leg_r_2_f1: geometry collision box size=0.05 0.07 0.05; visual mesh filename=package://hexapod_model/meshes/femur_1_bin.stl
- link leg_r_2_f2: geometry collision box size=0.11 0.03 0.06; visual mesh filename=package://hexapod_model/meshes/femur_3_bin.stl
- link leg_r_2_f3: geometry collision box size=0.12 0.03 0.06; visual mesh filename=package://hexapod_model/meshes/femur_2_bin.stl
- link leg_r_2_f4: geometry collision box size=0.08 0.03 0.06; visual mesh filename=package://hexapod_model/meshes/femur_4_bin.stl
- link leg_r_3_f1: geometry collision box size=0.05 0.07 0.05; visual mesh filename=package://hexapod_model/meshes/femur_1_bin.stl
- link leg_r_3_f2: geometry collision box size=0.11 0.03 0.06; visual mesh filename=package://hexapod_model/meshes/femur_3_bin.stl
- link leg_r_3_f3: geometry collision box size=0.12 0.03 0.06; visual mesh filename=package://hexapod_model/meshes/femur_2_bin.stl
- link leg_r_3_f4: geometry collision box size=0.08 0.03 0.06; visual mesh filename=package://hexapod_model/meshes/femur_4_bin.stl
Joints:
- removed joint joint__1_f1
- removed joint joint__1_f2
- removed joint joint__1_f3
- removed joint joint__1_f4
- added joint joint_l_1_end: type fixed, parent leg_l_1_f4, child leg_l_1_end, origin xyz=0 0.067 0.0 rpy=0 0 0
- added joint joint_l_2_end: type fixed, parent leg_l_2_f4, child leg_l_2_end, origin xyz=0 0.067 0.0 rpy=0 0 0
- added joint joint_l_3_end: type fixed, parent leg_l_3_f4, child leg_l_3_end, origin xyz=0 0.067 0.0 rpy=0 0 0
- added joint joint_r_1_end: type fixed, parent leg_r_1_f4, child leg_r_1_end, origin xyz=0 0.067 0.0 rpy=0 0 0
- added joint joint_r_1_f1: type revolute, parent base_link, child leg_r_1_f1, origin xyz=0.103 -0.07 0 rpy=0 0 -1.57079632679, axis 0 0 1, limit lower=-1.57079632679 upper=1.57079632679 effort=15 velocity=1.0
- added joint joint_r_1_f2: type revolute, parent leg_r_1_f1, child leg_r_1_f2, origin xyz=0.062 0.0 0.0 rpy=0 0 1.57079632679, axis 1 0 0, limit lower=-1.57079632679 upper=1.57079632679 effort=15 velocity=1.0
- added joint joint_r_1_f3: type revolute, parent leg_r_1_f2, child leg_r_1_f3, origin xyz=0.0 -0.094 0.0 rpy=0 -1.00530964915 1.57079632679, axis 0 1 0, limit lower=-1.57079632679 upper=1.57079632679 effort=15 velocity=1.0
- added joint joint_r_1_f4: type revolute, parent leg_r_1_f3, child leg_r_1_f4, origin xyz=-0.104 0.0 0.0 rpy=-0 0 1.57079632679, axis 1 0 0, limit lower=-1.57079632679 upper=1.57079632679 effort=15 velocity=1.0
- added joint joint_r_2_end: type fixed, parent leg_r_2_f4, child leg_r_2_end, origin xyz=0 0.067 0.0 rpy=0 0 0
- added joint joint_r_3_end: type fixed, parent leg_r_3_f4, child leg_r_3_end, origin xyz=0 0.067 0.0 rpy=0 0 0
- joint joint_l_1_f1: limit lower=-1.57 upper=1.57 effort=15 velocity=1.0 -> lower=-1.57079632679 upper=1.57079632679 effort=15 velocity=1.0; origin xyz=0.103 0.07 0 rpy=0 0 0.7 -> xyz=0.103 0.07 0 rpy=0 0 1.57079632679
- joint joint_l_1_f2: axis 0 1 0 -> 1 0 0; limit lower=-1.57 upper=1.57 effort=15 velocity=1.0 -> lower=-1.57079632679 upper=1.57079632679 effort=15 velocity=1.0; origin xyz=0.0 -0.094 0.0 rpy=0 -2.3 1.57 -> xyz=0.062 0.0 0.0 rpy=0 0 1.57079632679; parent leg_l_1_f3 -> leg_l_1_f1
- joint joint_l_1_f3: axis 1 0 0 -> 0 1 0; limit lower=-1.57 upper=1.57 effort=15 velocity=1.0 -> lower=-1.57079632679 upper=1.57079632679 effort=15 velocity=1.0; origin xyz=0.062 0.0 0.0 rpy=-1.1 0 1.57 -> xyz=0.0 -0.094 0.0 rpy=0 -1.00530964915 1.57079632679; parent leg_l_1_f1 -> leg_l_1_f2
- joint joint_l_1_f4: limit lower=-1.57 upper=1.57 effort=15 velocity=1.0 -> lower=-1.57079632679 upper=1.57079632679 effort=15 velocity=1.0; origin xyz=-0.104 0.0 0.0 rpy=-0.4 0 1.57 -> xyz=-0.104 0.0 0.0 rpy=-0 0 1.57079632679; parent leg_l_1_f2 -> leg_l_1_f3
- joint joint_l_2_f1: limit lower=-1.57 upper=1.57 effort=15 velocity=1.0 -> lower=-1.57079632679 upper=1.57079632679 effort=15 velocity=1.0; origin xyz=0.0 0.096 0 rpy=0 0 1.4 -> xyz=0.0 0.096 0 rpy=0 0 1.57079632679
- joint joint_l_2_f2: limit lower=-1.57 upper=1.57 effort=15 velocity=1.0 -> lower=-1.57079632679 upper=1.57079632679 effort=15 velocity=1.0; origin xyz=0.0 -0.094 0.0 rpy=0 -2.3 1.57 -> xyz=0.062 0.0 0.0 rpy=0 0 1.57079632679; parent leg_l_2_f3 -> leg_l_2_f1
- joint joint_l_2_f3: axis 1 0 0 -> 0 1 0; limit lower=-1.57 upper=1.57 effort=15 velocity=1.0 -> lower=-1.57079632679 upper=1.57079632679 effort=15 velocity=1.0; origin xyz=0.062 0.0 0.0 rpy=-1.1 0 1.57 -> xyz=0.0 -0.094 0.0 rpy=0 -1.00530964915 1.57079632679; parent leg_l_2_f1 -> leg_l_2_f2
- joint joint_l_2_f4: limit lower=-1.57 upper=1.57 effort=15 velocity=1.0 -> lower=-1.57079632679 upper=1.57079632679 effort=15 velocity=1.0; origin xyz=-0.104 0.0 0.0 rpy=-0.4 0 1.57 -> xyz=-0.104 0.0 0.0 rpy=-0 0 1.57079632679; parent leg_l_2_f2 -> leg_l_2_f3
- joint joint_l_3_f1: limit lower=-1.57 upper=1.57 effort=15 velocity=1.0 -> lower=-1.57079632679 upper=1.57079632679 effort=15 velocity=1.0; origin xyz=-0.09 0.083 0 rpy=0 0 2.1 -> xyz=-0.09 0.083 0 rpy=0 0 1.57079632679
- joint joint_l_3_f2: limit lower=-1.57 upper=1.57 effort=15 velocity=1.0 -> lower=-1.57079632679 upper=1.57079632679 effort=15 velocity=1.0; origin xyz=0.0 -0.094 0.0 rpy=0 -2.3 1.57 -> xyz=0.062 0.0 0.0 rpy=0 0 1.57079632679; parent leg_l_3_f3 -> leg_l_3_f1
- joint joint_l_3_f3: axis 1 0 0 -> 0 1 0; limit lower=-1.57 upper=1.57 effort=15 velocity=1.0 -> lower=-1.57079632679 upper=1.57079632679 effort=15 velocity=1.0; origin xyz=0.062 0.0 0.0 rpy=-1.1 0 1.57 -> xyz=0.0 -0.094 0.0 rpy=0 -1.00530964915 1.57079632679; parent leg_l_3_f1 -> leg_l_3_f2
- joint joint_l_3_f4: limit lower=-1.57 upper=1.57 effort=15 velocity=1.0 -> lower=-1.57079632679 upper=1.57079632679 effort=15 velocity=1.0; origin xyz=-0.104 0.0 0.0 rpy=-0.4 0 1.57 -> xyz=-0.104 0.0 0.0 rpy=-0 0 1.57079632679; parent leg_l_3_f2 -> leg_l_3_f3
- joint joint_r_2_f1: limit lower=-1.57 upper=1.57 effort=15 velocity=1.0 -> lower=-1.57079632679 upper=1.57079632679 effort=15 velocity=1.0; origin xyz=0.0 -0.096 0 rpy=0 0 -1.4 -> xyz=0.0 -0.096 0 rpy=0 0 -1.57079632679
- joint joint_r_2_f2: limit lower=-1.57 upper=1.57 effort=15 velocity=1.0 -> lower=-1.57079632679 upper=1.57079632679 effort=15 velocity=1.0; origin xyz=0.0 -0.094 0.0 rpy=0 -2.3 1.57 -> xyz=0.062 0.0 0.0 rpy=0 0 1.57079632679; parent leg_r_2_f3 -> leg_r_2_f1
- joint joint_r_2_f3: axis 1 0 0 -> 0 1 0; limit lower=-1.57 upper=1.57 effort=15 velocity=1.0 -> lower=-1.57079632679 upper=1.57079632679 effort=15 velocity=1.0; origin xyz=0.062 0.0 0.0 rpy=-1.1 0 1.57 -> xyz=0.0 -0.094 0.0 rpy=0 -1.00530964915 1.57079632679; parent leg_r_2_f1 -> leg_r_2_f2
- joint joint_r_2_f4: limit lower=-1.57 upper=1.57 effort=15 velocity=1.0 -> lower=-1.57079632679 upper=1.57079632679 effort=15 velocity=1.0; origin xyz=-0.104 0.0 0.0 rpy=-0.4 0 1.57 -> xyz=-0.104 0.0 0.0 rpy=-0 0 1.57079632679; parent leg_r_2_f2 -> leg_r_2_f3
- joint joint_r_3_f1: limit lower=-1.57 upper=1.57 effort=15 velocity=1.0 -> lower=-1.57079632679 upper=1.57079632679 effort=15 velocity=1.0; origin xyz=-0.09 -0.083 0 rpy=0 0 -2.1 -> xyz=-0.09 -0.083 0 rpy=0 0 -1.57079632679
- joint joint_r_3_f2: limit lower=-1.57 upper=1.57 effort=15 velocity=1.0 -> lower=-1.57079632679 upper=1.57079632679 effort=15 velocity=1.0; origin xyz=0.0 -0.094 0.0 rpy=0 -2.3 1.57 -> xyz=0.062 0.0 0.0 rpy=0 0 1.57079632679; parent leg_r_3_f3 -> leg_r_3_f1
- joint joint_r_3_f3: axis 1 0 0 -> 0 1 0; limit lower=-1.57 upper=1.57 effort=15 velocity=1.0 -> lower=-1.57079632679 upper=1.57079632679 effort=15 velocity=1.0; origin xyz=0.062 0.0 0.0 rpy=-1.1 0 1.57 -> xyz=0.0 -0.094 0.0 rpy=0 -1.00530964915 1.57079632679; parent leg_r_3_f1 -> leg_r_3_f2
- joint joint_r_3_f4: limit lower=-1.57 upper=1.57 effort=15 velocity=1.0 -> lower=-1.57079632679 upper=1.57079632679 effort=15 velocity=1.0; origin xyz=-0.104 0.0 0.0 rpy=-0.4 0 1.57 -> xyz=-0.104 0.0 0.0 rpy=-0 0 1.57079632679; parent leg_r_3_f2 -> leg_r_3_f3

File: src/hexapod_model/urdf/hexapod.xacro (robot description, xacro)
@@ -1,137 +1,2 @@
 <?xml version="1.0" encoding="US-ASCII"?>
-<robot name="hexapod" xmlns:xacro="http://www.ros.org/wiki/xacro">
-	<xacro:property name="pi" value="3.1415926535897931" />
-	<link name="base_link">
-		<visual>
-			<origin rpy="${0.5 * pi} 0 0"/>
-			<geometry>
-				<mesh filename="package://hexapod_model/meshes/body_bin.stl"/>
-			</geometry>
-			<material name="abs">
-				<color rgba="0.6 0.6 0.6 1"/>
-			</material>
-			<collision>
-				<origin rpy="${0.5 * pi} 0 0"/>
-				<geometry>
-					<mesh filename="package://hexapod_model/meshes/body_bin.stl"/>
-				</geometry>
-			</collision>
-		</visual>
-	</link>
-	<xacro:macro name="leg" params="side num *origin">
-		<link name="leg_${side}_${num}_f1">
-			<visual>
-				<origin rpy="0 ${0.5 * pi} -${0.5 * pi}" xyz="-0.009 0 0"/>
-				<geometry>
-					<mesh filename="package://hexapod_model/meshes/femur_1_bin.stl"/>
-				</geometry>
-				<material name="abs1">
-					<color rgba="0.9 0.0 0.0 1" />
-				</material>
-				<collision>
-					<origin rpy="0 ${0.5 * pi} -${0.5 * pi}" xyz="-0.009 0 0"/>
-					<geometry>
-						<mesh filename="package://hexapod_model/meshes/femur_1_bin.stl"/>
-					</geometry>
-				</collision>
-			</visual>
-		</link>
-		<link name="leg_${side}_${num}_f2">
-			<visual>
-				<origin rpy="${1.5 * pi} 0 ${0.5 * pi}" xyz="0 -0.053 0.013"/>
-				<geometry>
-					<mesh filename="package://hexapod_model/meshes/femur_3_bin.stl"/>
-				</geometry>
-				<material name="abs2">
-					<color rgba="0.0 0.9 0.0 1"/>
-				</material>
-				<collision>
-					<origin rpy="${1.5 * pi} 0 ${0.5 * pi}" xyz="0 -0.053 0.013"/>
-					<geometry>
-						<mesh filename="package://hexapod_model/meshes/femur_3_bin.stl"/>
-					</geometry>
-				</collision>
-			</visual>
-		</link>
-		<link name="leg_${side}_${num}_f3">
-			<visual>
-				<origin rpy="${1.5 * pi} 0 0" xyz="-0.063 0 0.013"/>
-				<geometry>
-					<mesh filename="package://hexapod_model/meshes/femur_2_bin.stl"/>
-				</geometry>
-				<material name="abs3">
-					<color rgba="0.0 0.0 0.9 1"/>
-				</material>
-				<collision>
-					<origin rpy="${1.5 * pi} 0 0" xyz="-0.063 0 0.013"/>
-					<geometry>
-						<mesh filename="package://hexapod_model/meshes/femur_2_bin.stl"/>
-					</geometry>
-				</collision>
-			</visual>
-		</link>
-		<link name="leg_${side}_${num}_f4">
-			<visual>
-				<origin rpy="${0.5 * pi} 0 ${1.5 * pi}" xyz="0 0.038 -0.013"/>
-				<geometry>
-					<mesh filename="package://hexapod_model/meshes/femur_4_bin.stl"/>
-				</geometry>
-				<material name="abs4">
-					<color rgba="0.8 0.8 0.0 1"/>
-				</material>
-				<collision>
-					<origin rpy="${0.5 * pi} 0 ${1.5 * pi}" xyz="0 0.038 -0.013"/>
-					<geometry>
-						<mesh filename="package://hexapod_model/meshes/femur_4_bin.stl"/>
-					</geometry>
-				</collision>
-			</visual>
-		</link>
-		<joint name="joint_${side}_${num}_f1" type="revolute">
-			<parent link="base_link"/>
-			<child link="leg_${side}_${num}_f1"/>
-			<xacro:insert_block name="origin" />
-			<axis xyz="0 0 1" />
-			<limit lower="-${0.5 * pi}" upper="${0.5 * pi}" effort="15" velocity="1.0" />
-	  	</joint>
-		<joint name="joint_${side}_${num}_f2" type="revolute">
-			<parent link="leg_${side}_${num}_f1"/>
-			<child link="leg_${side}_${num}_f2"/>
-			<origin xyz="0.062 0.0 0.0" rpy="0 0 ${0.5 * pi}" />
-			<axis xyz="1 0 0" />
-			<limit lower="-${0.5 * pi}" upper="${0.5 * pi}" effort="15" velocity="1.0" />
-	  	</joint>
-		<joint name="joint_${side}_${num}_f3" type="revolute">
-			<parent link="leg_${side}_${num}_f2"/>
-			<child link="leg_${side}_${num}_f3"/>
-			<origin xyz="0.0 -0.094 0.0" rpy="0 -${0.32 * pi} ${0.5 * pi}" />
-			<axis xyz="0 1 0" />
-			<limit lower="-${0.5 * pi}" upper="${0.5 * pi}" effort="15" velocity="1.0" />
-	  	</joint>
-		<joint name="joint_${side}_${num}_f4" type="revolute">
-			<parent link="leg_${side}_${num}_f3"/>
-			<child link="leg_${side}_${num}_f4"/>
-			<origin xyz="-0.104 0.0 0.0" rpy="-0 0 ${0.5 * pi}" />
-			<axis xyz="1 0 0" />
-			<limit lower="-${0.5 * pi}" upper="${0.5 * pi}" effort="15" velocity="1.0" />
-	  	</joint>
-	</xacro:macro>
-	<xacro:leg side="l" num="1">
-		<origin xyz="0.103 0.07 0" rpy="0 0 ${0.5 * pi}" />
-	</xacro:leg>
-	<xacro:leg side="l" num="2">
-		<origin xyz="0.0 0.096 0" rpy="0 0 ${0.5 * pi}" />
-	</xacro:leg>
-	<xacro:leg side="l" num="3">
-		<origin xyz="-0.09 0.083 0" rpy="0 0 ${0.5 * pi}" />
-	</xacro:leg>
-	<xacro:leg side="r" num="1">
-		<origin xyz="0.103 -0.07 0" rpy="0 0 -${0.5 * pi}" />
-	</xacro:leg>
-	<xacro:leg side="r" num="2">
-		<origin xyz="0.0 -0.096 0" rpy="0 0 -${0.5 * pi}" />
-	</xacro:leg>
-	<xacro:leg side="r" num="3">
-		<origin xyz="-0.09 -0.083 0" rpy="0 0 -${0.5 * pi}" />
-	</xacro:leg>
-</robot>
+<robot xmlns:xacro="http://www.ros.org/wiki/xacro" name="hexapod"><xacro:property name="pi" value="3.1415926535897931"/><link name="base_link"><visual><origin rpy="${0.5 * pi} 0 0"/><geometry><mesh filename="package://hexapod_model/meshes/body_bin.stl"/></geometry><material name="abs"><color rgba="0.6 0.6 0.6 1"/></material></visual><collision><origin rpy="${0.5 * pi} 0 0"/><geometry><box size="0.19 0.05 0.14"/></geometry></collision></link><xacro:macro name="leg" params="side num *origin"><link name="leg_${side}_${num}_f1"><visual><origin rpy="0 ${0.5 * pi} -${0.5 * pi}" xyz="-0.009 0 0"/><geometry><mesh filename="package://hexapod_model/meshes/femur_1_bin.stl"/></geometry><material name="abs1"><color rgba="0.9 0.0 0.0 1"/></material></visual><collision><origin rpy="0 ${0.5 * pi} -${0.5 * pi}" xyz="0.04 0 0"/><geometry><box size="0.05 0.07 0.05"/></geometry></collision></link><link name="leg_${side}_${num}_f2"><visual><origin rpy="${1.5 * pi} 0 ${0.5 * pi}" xyz="0 -0.053 0.013"/><geometry><mesh filename="package://hexapod_model/meshes/femur_3_bin.stl"/></geometry><material name="abs2"><color rgba="0.0 0.9 0.0 1"/></material></visual><collision><origin rpy="${1.5 * pi} 0 ${0.5 * pi}" xyz="0 -0.043 0"/><geometry><box size="0.11 0.03 0.06"/></geometry></collision></link><link name="leg_${side}_${num}_f3"><visual><origin rpy="${1.5 * pi} 0 0" xyz="-0.063 0 0.013"/><geometry><mesh filename="package://hexapod_model/meshes/femur_2_bin.stl"/></geometry><material name="abs3"><color rgba="0.0 0.0 0.9 1"/></material></visual><collision><origin rpy="${1.5 * pi} 0 0" xyz="-0.043 0 0"/><geometry><box size="0.12 0.03 0.06"/></geometry></collision></link><link name="leg_${side}_${num}_f4"><visual><origin rpy="${0.5 * pi} 0 ${1.5 * pi}" xyz="0 0.038 -0.013"/><geometry><mesh filename="package://hexapod_model/meshes/femur_4_bin.stl"/></geometry><material name="abs4"><color rgba="0.8 0.8 0.0 1"/></material></visual><collision><origin rpy="${0.5 * pi} 0 ${1.5 * pi}" xyz="0 0.028 0"/><geometry><box size="0.08 0.03 0.06"/></geometry></collision></link><link name="leg_${side}_${num}_end"><visual><geometry><box size="0.02 0.005 0.02 "/></geometry><material name="abs_end"><color rgba="1 1 1 1"/></material></visual><collision><geometry><box size="0.02 0.005 0.02 "/></geometry></collision></link><joint name="joint_${side}_${num}_f1" type="revolute"><parent link="base_link"/><child link="leg_${side}_${num}_f1"/><xacro:insert_block name="origin"/><axis xyz="0 0 1"/><limit lower="-${0.5 * pi}" upper="${0.5 * pi}" effort="15" velocity="1.0"/></joint><joint name="joint_${side}_${num}_f2" type="revolute"><parent link="leg_${side}_${num}_f1"/><child link="leg_${side}_${num}_f2"/><origin xyz="0.062 0.0 0.0" rpy="0 0 ${0.5 * pi}"/><axis xyz="1 0 0"/><limit lower="-${0.5 * pi}" upper="${0.5 * pi}" effort="15" velocity="1.0"/></joint><joint name="joint_${side}_${num}_f3" type="revolute"><parent link="leg_${side}_${num}_f2"/><child link="leg_${side}_${num}_f3"/><origin xyz="0.0 -0.094 0.0" rpy="0 -${0.32 * pi} ${0.5 * pi}"/><axis xyz="0 1 0"/><limit lower="-${0.5 * pi}" upper="${0.5 * pi}" effort="15" velocity="1.0"/></joint><joint name="joint_${side}_${num}_f4" type="revolute"><parent link="leg_${side}_${num}_f3"/><child link="leg_${side}_${num}_f4"/><origin xyz="-0.104 0.0 0.0" rpy="-0 0 ${0.5 * pi}"/><axis xyz="1 0 0"/><limit lower="-${0.5 * pi}" upper="${0.5 * pi}" effort="15" velocity="1.0"/></joint><joint name="joint_${side}_${num}_end" type="fixed"><parent link="leg_${side}_${num}_f4"/><child link="leg_${side}_${num}_end"/><origin xyz="0 0.067 0.0" rpy="0 0 0"/></joint></xacro:macro><xacro:leg side="l" num="1"><origin xyz="0.103 0.07 0" rpy="0 0 ${0.5 * pi}"/></xacro:leg><xacro:leg side="l" num="2"><origin xyz="0.0 0.096 0" rpy="0 0 ${0.5 * pi}"/></xacro:leg><xacro:leg side="l" num="3"><origin xyz="-0.09 0.083 0" rpy="0 0 ${0.5 * pi}"/></xacro:leg><xacro:leg side="r" num="1"><origin xyz="0.103 -0.07 0" rpy="0 0 -${0.5 * pi}"/></xacro:leg><xacro:leg side="r" num="2"><origin xyz="0.0 -0.096 0" rpy="0 0 -${0.5 * pi}"/></xacro:leg><xacro:leg side="r" num="3"><origin xyz="-0.09 -0.083 0" rpy="0 0 -${0.5 * pi}"/></xacro:leg></robot>
