Commit message: fix of initial leg positions

File: src/hexapod_model/urdf/hexapod.urdf (robot description, URDF)
Before this commit: robot hexapod, 31 links, 30 joints
Joints:
- joint joint_l_1_f1: origin xyz=0.103 0.07 0 rpy=0 0 1.57079632679 -> xyz=0.103 0.07 0 rpy=0 0 0.69115038379
- joint joint_l_3_f1: origin xyz=-0.09 0.083 0 rpy=0 0 1.57079632679 -> xyz=-0.09 0.083 0 rpy=0 0 2.10486707791
- joint joint_r_1_f1: origin xyz=0.103 -0.07 0 rpy=0 0 -1.57079632679 -> xyz=0.103 -0.07 0 rpy=0 0 -0.69115038379
- joint joint_r_3_f1: origin xyz=-0.09 -0.083 0 rpy=0 0 -1.57079632679 -> xyz=-0.09 -0.083 0 rpy=0 0 -2.10486707791

File: src/hexapod_model/urdf/hexapod.xacro (robot description, xacro)
@@ -1,2 +1,161 @@
-<?xml version="1.0" encoding="US-ASCII"?>
-<robot xmlns:xacro="http://www.ros.org/wiki/xacro" name="hexapod"><xacro:property name="pi" value="3.1415926535897931"/><link name="base_link"><visual><origin rpy="${0.5 * pi} 0 0"/><geometry><mesh filename="package://hexapod_model/meshes/body_bin.stl"/></geometry><material name="abs"><color rgba="0.6 0.6 0.6 1"/></material></visual><collision><origin rpy="${0.5 * pi} 0 0"/><geometry><box size="0.19 0.05 0.14"/></geometry></collision></link><xacro:macro name="leg" params="side num *origin"><link name="leg_${side}_${num}_f1"><visual><origin rpy="0 ${0.5 * pi} -${0.5 * pi}" xyz="-0.009 0 0"/><geometry><mesh filename="package://hexapod_model/meshes/femur_1_bin.stl"/></geometry><material name="abs1"><color rgba="0.9 0.0 0.0 1"/></material></visual><collision><origin rpy="0 ${0.5 * pi} -${0.5 * pi}" xyz="0.04 0 0"/><geometry><box size="0.05 0.07 0.05"/></geometry></collision></link><link name="leg_${side}_${num}_f2"><visual><origin rpy="${1.5 * pi} 0 ${0.5 * pi}" xyz="0 -0.053 0.013"/><geometry><mesh filename="package://hexapod_model/meshes/femur_3_bin.stl"/></geometry><material name="abs2"><color rgba="0.0 0.9 0.0 1"/></material></visual><collision><origin rpy="${1.5 * pi} 0 ${0.5 * pi}" xyz="0 -0.043 0"/><geometry><box size="0.11 0.03 0.06"/></geometry></collision></link><link name="leg_${side}_${num}_f3"><visual><origin rpy="${1.5 * pi} 0 0" xyz="-0.063 0 0.013"/><geometry><mesh filename="package://hexapod_model/meshes/femur_2_bin.stl"/></geometry><material name="abs3"><color rgba="0.0 0.0 0.9 1"/></material></visual><collision><origin rpy="${1.5 * pi} 0 0" xyz="-0.043 0 0"/><geometry><box size="0.12 0.03 0.06"/></geometry></collision></link><link name="leg_${side}_${num}_f4"><visual><origin rpy="${0.5 * pi} 0 ${1.5 * pi}" xyz="0 0.038 -0.013"/><geometry><mesh filename="package://hexapod_model/meshes/femur_4_bin.stl"/></geometry><material name="abs4"><color rgba="0.8 0.8 0.0 1"/></material></visual><collision><origin rpy="${0.5 * pi} 0 ${1.5 * pi}" xyz="0 0.028 0"/><geometry><box size="0.08 0.03 0.06"/></geometry></collision></link><link name="leg_${side}_${num}_end"><visual><geometry><box size="0.02 0.005 0.02 "/></geometry><material name="abs_end"><color rgba="1 1 1 1"/></material></visual><collision><geometry><box size="0.02 0.005 0.02 "/></geometry></collision></link><joint name="joint_${side}_${num}_f1" type="revolute"><parent link="base_link"/><child link="leg_${side}_${num}_f1"/><xacro:insert_block name="origin"/><axis xyz="0 0 1"/><limit lower="-${0.5 * pi}" upper="${0.5 * pi}" effort="15" velocity="1.0"/></joint><joint name="joint_${side}_${num}_f2" type="revolute"><parent link="leg_${side}_${num}_f1"/><child link="leg_${side}_${num}_f2"/><origin xyz="0.062 0.0 0.0" rpy="0 0 ${0.5 * pi}"/><axis xyz="1 0 0"/><limit lower="-${0.5 * pi}" upper="${0.5 * pi}" effort="15" velocity="1.0"/></joint><joint name="joint_${side}_${num}_f3" type="revolute"><parent link="leg_${side}_${num}_f2"/><child link="leg_${side}_${num}_f3"/><origin xyz="0.0 -0.094 0.0" rpy="0 -${0.32 * pi} ${0.5 * pi}"/><axis xyz="0 1 0"/><limit lower="-${0.5 * pi}" upper="${0.5 * pi}" effort="15" velocity="1.0"/></joint><joint name="joint_${side}_${num}_f4" type="revolute"><parent link="leg_${side}_${num}_f3"/><child link="leg_${side}_${num}_f4"/><origin xyz="-0.104 0.0 0.0" rpy="-0 0 ${0.5 * pi}"/><axis xyz="1 0 0"/><limit lower="-${0.5 * pi}" upper="${0.5 * pi}" effort="15" velocity="1.0"/></joint><joint name="joint_${side}_${num}_end" type="fixed"><parent link="leg_${side}_${num}_f4"/><child link="leg_${side}_${num}_end"/><origin xyz="0 0.067 0.0" rpy="0 0 0"/></joint></xacro:macro><xacro:leg side="l" num="1"><origin xyz="0.103 0.07 0" rpy="0 0 ${0.5 * pi}"/></xacro:leg><xacro:leg side="l" num="2"><origin xyz="0.0 0.096 0" rpy="0 0 ${0.5 * pi}"/></xacro:leg><xacro:leg side="l" num="3"><origin xyz="-0.09 0.083 0" rpy="0 0 ${0.5 * pi}"/></xacro:leg><xacro:leg side="r" num="1"><origin xyz="0.103 -0.07 0" rpy="0 0 -${0.5 * pi}"/></xacro:leg><xacro:leg side="r" num="2"><origin xyz="0.0 -0.096 0" rpy="0 0 -${0.5 * pi}"/></xacro:leg><xacro:leg side="r" num="3"><origin xyz="-0.09 -0.083 0" rpy="0 0 -${0.5 * pi}"/></xacro:leg></robot>
+<?xml version="1.0" ?>
+<robot xmlns:xacro="http://www.ros.org/wiki/xacro" name="hexapod">
+	<xacro:property name="pi" value="3.1415926535897931" />
+	<link name="base_link">
+		<visual>
+			<origin rpy="${0.5 * pi} 0 0" />
+			<geometry>
+				<mesh filename="package://hexapod_model/meshes/body_bin.stl" />
+			</geometry>
+			<material name="abs">
+				<color rgba="0.6 0.6 0.6 1" />
+			</material>
+		</visual>
+		<collision>
+			<origin rpy="${0.5 * pi} 0 0" />
+			<geometry>
+				<box size="0.19 0.05 0.14" />
+			</geometry>
+		</collision>
+	</link>
+	<xacro:macro name="leg" params="side num *origin">
+		<link name="leg_${side}_${num}_f1">
+			<visual>
+				<origin rpy="0 ${0.5 * pi} -${0.5 * pi}" xyz="-0.009 0 0" />
+				<geometry>
+					<mesh filename="package://hexapod_model/meshes/femur_1_bin.stl" />
+				</geometry>
+				<material name="abs1">
+					<color rgba="0.9 0.0 0.0 1" />
+				</material>
+			</visual>
+			<collision>
+				<origin rpy="0 ${0.5 * pi} -${0.5 * pi}" xyz="0.04 0 0" />
+				<geometry>
+					<box size="0.05 0.07 0.05" />
+				</geometry>
+			</collision>
+		</link>
+		<link name="leg_${side}_${num}_f2">
+			<visual>
+				<origin rpy="${1.5 * pi} 0 ${0.5 * pi}" xyz="0 -0.053 0.013" />
+				<geometry>
+					<mesh filename="package://hexapod_model/meshes/femur_3_bin.stl" />
+				</geometry>
+				<material name="abs2">
+					<color rgba="0.0 0.9 0.0 1" />
+				</material>
+			</visual>
+			<collision>
+				<origin rpy="${1.5 * pi} 0 ${0.5 * pi}" xyz="0 -0.043 0" />
+				<geometry>
+					<box size="0.11 0.03 0.06" />
+				</geometry>
+			</collision>
+		</link>
+		<link name="leg_${side}_${num}_f3">
+			<visual>
+				<origin rpy="${1.5 * pi} 0 0" xyz="-0.063 0 0.013" />
+				<geometry>
+					<mesh filename="package://hexapod_model/meshes/femur_2_bin.stl" />
+				</geometry>
+				<material name="abs3">
+					<color rgba="0.0 0.0 0.9 1" />
+				</material>
+			</visual>
+			<collision>
+				<origin rpy="${1.5 * pi} 0 0" xyz="-0.043 0 0" />
+				<geometry>
+					<box size="0.12 0.03 0.06" />
+				</geometry>
+			</collision>
+		</link>
+		<link name="leg_${side}_${num}_f4">
+			<visual>
+				<origin rpy="${0.5 * pi} 0 ${1.5 * pi}" xyz="0 0.038 -0.013" />
+				<geometry>
+					<mesh filename="package://hexapod_model/meshes/femur_4_bin.stl" />
+				</geometry>
+				<material name="abs4">
+					<color rgba="0.8 0.8 0.0 1" />
+				</material>
+			</visual>
+			<collision>
+				<origin rpy="${0.5 * pi} 0 ${1.5 * pi}" xyz="0 0.028 0" />
+				<geometry>
+					<box size="0.08 0.03 0.06" />
+				</geometry>
+			</collision>
+		</link>
+		<link name="leg_${side}_${num}_end">
+			<visual>
+				<geometry>
+					<box size="0.02 0.005 0.02 " />
+				</geometry>
+				<material name="abs_end">
+					<color rgba="1 1 1 1" />
+				</material>
+			</visual>
+			<collision>
+				<geometry>
+					<box size="0.02 0.005 0.02 " />
+				</geometry>
+			</collision>
+		</link>
+		<joint name="joint_${side}_${num}_f1" type="revolute">
+			<parent link="base_link" />
+			<child link="leg_${side}_${num}_f1" />
+			<xacro:insert_block name="origin" />
+			<axis xyz="0 0 1" />
+			<limit lower="-${0.5 * pi}" upper="${0.5 * pi}" effort="15"
+				velocity="1.0" />
+		</joint>
+		<joint name="joint_${side}_${num}_f2" type="revolute">
+			<parent link="leg_${side}_${num}_f1" />
+			<child link="leg_${side}_${num}_f2" />
+			<origin xyz="0.062 0.0 0.0" rpy="0 0 ${0.5 * pi}" />
+			<axis xyz="1 0 0" />
+			<limit lower="-${0.5 * pi}" upper="${0.5 * pi}" effort="15"
+				velocity="1.0" />
+		</joint>
+		<joint name="joint_${side}_${num}_f3" type="revolute">
+			<parent link="leg_${side}_${num}_f2" />
+			<child link="leg_${side}_${num}_f3" />
+			<origin xyz="0.0 -0.094 0.0" rpy="0 -${0.32 * pi} ${0.5 * pi}" />
+			<axis xyz="0 1 0" />
+			<limit lower="-${0.5 * pi}" upper="${0.5 * pi}" effort="15"
+				velocity="1.0" />
+		</joint>
+		<joint name="joint_${side}_${num}_f4" type="revolute">
+			<parent link="leg_${side}_${num}_f3" />
+			<child link="leg_${side}_${num}_f4" />
+			<origin xyz="-0.104 0.0 0.0" rpy="-0 0 ${0.5 * pi}" />
+			<axis xyz="1 0 0" />
+			<limit lower="-${0.5 * pi}" upper="${0.5 * pi}" effort="15"
+				velocity="1.0" />
+		</joint>
+		<joint name="joint_${side}_${num}_end" type="fixed">
+			<parent link="leg_${side}_${num}_f4" />
+			<child link="leg_${side}_${num}_end" />
+			<origin xyz="0 0.067 0.0" rpy="0 0 0" />
+		</joint>
+	</xacro:macro>
+	<xacro:leg side="l" num="1">
+		<origin xyz="0.103 0.07 0" rpy="0 0 ${0.22 * pi}" />
+	</xacro:leg>
+	<xacro:leg side="l" num="2">
+		<origin xyz="0.0 0.096 0" rpy="0 0 ${0.5 * pi}" />
+	</xacro:leg>
+	<xacro:leg side="l" num="3">
+		<origin xyz="-0.09 0.083 0" rpy="0 0 ${0.67 * pi}" />
+	</xacro:leg>
+	<xacro:leg side="r" num="1">
+		<origin xyz="0.103 -0.07 0" rpy="0 0 -${0.22 * pi}" />
+	</xacro:leg>
+	<xacro:leg side="r" num="2">
+		<origin xyz="0.0 -0.096 0" rpy="0 0 -${0.5 * pi}" />
+	</xacro:leg>
+	<xacro:leg side="r" num="3">
+		<origin xyz="-0.09 -0.083 0" rpy="0 0 -${0.67 * pi}" />
+	</xacro:leg>
+</robot>
